File: FOC/MCU.kicad_sch (KiCad schematic)
At the start: 32 parts, among them J1 Conn_ARM_JTAG_SWD_10, SW1 SW_Push, SW2 SW_Push, U1 STM32G431CBTx, U3 SN65HVD230, Y1 Crystal_GND24

Commit message: CAN + UART done;driver controller done
Parts:
- added J3: UART_debug, Connector_PinHeader_2.54mm:PinHeader_1x03_P2.54mm_Vertical, symbol Connector:Conn_01x03_Socket
- C1, C14, C2, C3: renamed from C?; footprint (none) -> Capacitor_SMD:C_0603_1608Metric
- C10: renamed from C9; footprint (none) -> Capacitor_SMD:C_0603_1608Metric
- C11: renamed from C2; footprint (none) -> Capacitor_SMD:C_0603_1608Metric
- C12: renamed from C3; footprint (none) -> Capacitor_SMD:C_0603_1608Metric
- C13: renamed from C1; footprint (none) -> Capacitor_SMD:C_0603_1608Metric
- C4: renamed from C10; footprint (none) -> Capacitor_SMD:C_0603_1608Metric
- C5: footprint (none) -> Capacitor_SMD:C_0603_1608Metric
- C6: renamed from C4; footprint (none) -> Capacitor_SMD:C_0603_1608Metric
- C7: renamed from C6; footprint (none) -> Capacitor_SMD:C_0603_1608Metric
- C8: renamed from C7; footprint (none) -> Capacitor_SMD:C_0603_1608Metric
- C9: renamed from C8; footprint (none) -> Capacitor_SMD:C_0603_1608Metric
- D1: renamed from D3; footprint (none) -> LED_SMD:LED_0603_1608Metric
- D2: footprint (none) -> LED_SMD:LED_0603_1608Metric
- D3: renamed from D4; footprint (none) -> LED_SMD:LED_0603_1608Metric
- FB1: footprint (none) -> Inductor_SMD:L_0603_1608Metric
- J1: renamed from J?; footprint (none) -> Connector_JST:JST_SH_SM06B-SRSS-TB_1x06-1MP_P1.00mm_Horizontal
- J2: renamed from J1; footprint (none) -> Connector_PinHeader_1.27mm:PinHeader_2x05_P1.27mm_Vertical_SMD
- JP1: renamed from JP?; footprint (none) -> Jumper:SolderJumper-2_P1.3mm_Bridged_RoundedPad1.0x1.5mm
- R1: renamed from R3; footprint (none) -> Resistor_SMD:R_0603_1608Metric
- R2: footprint (none) -> Resistor_SMD:R_0603_1608Metric
- R3: renamed from R4; footprint (none) -> Resistor_SMD:R_0603_1608Metric
- R4: renamed from R1; footprint (none) -> Resistor_SMD:R_0603_1608Metric
- R5, R6: renamed from R?; footprint (none) -> Resistor_SMD:R_0603_1608Metric
- SW1: renamed from SW2; footprint (none) -> Button_Switch_SMD:SW_SPST_B3S-1000
- SW2: renamed from SW1; footprint (none) -> Button_Switch_SMD:SW_SPST_B3S-1000
- Y1: footprint (none) -> Crystal:Crystal_SMD_3225-4Pin_3.2x2.5mm
- renumbered U3 to U2
Connections:
- net GND: now also J3.3 (Pin_3)
- net UART_RX: now also J3.2 (Pin_2)
- net UART_TX: now also J3.1 (Pin_1); no longer C4.2, J2.10 (~{RESET}), SW2.1, U1.7 (PG10)
- new net RESET: C4.2, J2.10 (~{RESET}), SW2.1, U1.7 (PG10)
- no-connect marks 3 -> 13
Other:
- moved on the sheet: C11, C12, C13, FB1
