File: FOC/FOC.kicad_pcb (KiCad board)
At the start: 4 copper layers, 79 x 34.9 mm, 79 parts, among them J1 encoder_conn, J2 Conn_ARM_JTAG_SWD_10, J3 UART_debug, J4 XT30PW-M, J5 Conn_01x04_Socket, J6 Conn_01x04_Socket, J7 Conn_01x03_Socket, SW1 SW_Push, SW2 SW_Push, U1 STM32G431CBTx, U2 SN65HVD230, U3 TPS54202DDC, U4 AP2112K-3.3, U5 DRV8313PWP, Y1 Crystal_GND24

Commit message: drc erc clean; ready to order
Parts:
- moved D3 0.46 mm to (180.8, 98.7)
- moved R3 0.38 mm to (183.2, 99.5)
Routing:
- net GND: track 65.8 -> 40.0 mm, vias 30 -> 21
- net VM: track 85.4 -> 95.0 mm
