File: FOC/_restore_backup_2026-07-22T00-53-55-408/MCU.kicad_sch (KiCad schematic)
At the start: 33 parts, among them J1 encoder_conn, J2 Conn_ARM_JTAG_SWD_10, J3 UART_debug, SW1 SW_Push, SW2 SW_Push, U1 STM32G431CBTx, U2 SN65HVD230, Y1 Crystal_GND24

Commit message: four layer pour; layout done
Parts:
- J3: footprint Connector_PinSocket_2.54mm:PinSocket_1x03_P2.54mm_Vertical -> Connector_PinHeader_2.54mm:PinHeader_1x03_P2.54mm_Vertical
Changed lines of the file:
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@@
 			)
 		)
-		(property "Footprint" "Connector_PinSocket_2.54mm:PinSocket_1x03_P2.54mm_Vertical"
+		(property "Footprint" "Connector_PinHeader_2.54mm:PinHeader_1x03_P2.54mm_Vertical"
 			(at 234.95 77.47 0)
 			(hide yes)
